File: KiCad/AmigaDualFloppyInterface.kicad_sch (KiCad schematic)
At the start: 20 parts, among them J1 Floppy Power In, J2 Floppy B, J3 Motherboard, J4 Floppy Power Out, J5 Floppy A, J6 Conn_01x02_Pin, J7 Conn_01x02_Pin, U1 74LS38, U2 74LS74, U3 74LS157

Commit message: Add files via upload
Updated design with separate df1 LED
Parts:
- added J8: DF1 Activity, Connector_PinHeader_2.54mm:PinHeader_1x02_P2.54mm_Horizontal, symbol Connector:Conn_01x02_Pin
- added Q1: 2N3906, Package_TO_SOT_THT:TO-92_Inline, symbol Transistor_BJT:2N3906
- added R8: 4.7k, Resistor_THT:R_Axial_DIN0207_L6.3mm_D2.5mm_P7.62mm_Horizontal, symbol Device:R
- C1, C2, C3: footprint Capacitor_THT:C_Disc_D3.0mm_W2.0mm_P2.50mm -> Capacitor_THT:C_Disc_D4.3mm_W1.9mm_P5.00mm
- J6: value Conn_01x02_Pin -> Drive Switch
- R1, R2, R3, R4, R5, R7: footprint Resistor_THT:R_Axial_DIN0204_L3.6mm_D1.6mm_P5.08mm_Horizontal -> Resistor_THT:R_Axial_DIN0207_L6.3mm_D2.5mm_P7.62mm_Horizontal
- R6: value 1k -> 10k; footprint Resistor_THT:R_Axial_DIN0204_L3.6mm_D1.6mm_P5.08mm_Horizontal -> Resistor_THT:R_Axial_DIN0207_L6.3mm_D2.5mm_P7.62mm_Horizontal
Connections:
- net GND: now also U1.10, U1.12, U1.13, U1.9, J8.1 (Pin_1)
- net VCC: now also Q1.3 (C)
- net ~{MTR1}: now also R6.2, R8.1
- net ~{MTRA}: no longer U1.9
- net ~{MTRB}: no longer U1.10
- net ~{INUSE}: no longer names the net of U1.11
- net ~{INUSE}: no longer J3.4 (Pin_4)
- new net: J8.2 (Pin_2), Q1.1 (E)
- new net: Q1.2 (B), R8.2
- now unconnected: U1.8
- no-connect marks 14 -> 17
Other:
- note added: "DF1 Activity"
- note added: "Selection"
- note added: "Switching"
- note removed: "Floppy Lamp"
- note removed: "Phase 1"
- note removed: "Phase 2"
- note removed: "Phase 3"
- moved on the sheet: C3, J6, R7, U1C, U1D, U3
